Commit message: Full project upload: firmware, CAD scripts, docs, ROS2, PWA
Complete Mars Rover garden robot project for collaboration:
- 25 engineering analysis docs (EA-00 through EA-25)
- ESP32-S3 firmware (9 headers, compiles, 42 tests passing)
- 30 Fusion 360 CAD scripts (wheels, suspension, body, steering)
- 7 ROS2 packages (nav, perception, autonomy, teleop)
- Catppuccin Mocha PWA phone controller
- 3D print STLs (steering, suspension, wheels)
- CI/CD pipeline, wiring diagrams, BOM, build guides
- Custom Claude Code skills and commands

Co-Authored-By: Claude Opus 4.6 <noreply@anthropic.com>

File: software/jetson/rover_bringup/urdf/rover.urdf.xacro (robot description, xacro)
@@ -47,12 +47,12 @@
   <xacro:property name="rocker_pivot_x"   value="0.125" />  <!-- body pivot X offset -->
   <xacro:property name="rocker_pivot_z"   value="0.060" />  <!-- body pivot Z (at body bottom) -->
-  <!-- Bogie arms: 120mm total, pivot in middle -->
-  <xacro:property name="bogie_length"     value="0.120" />
+  <!-- Bogie arms: 180mm total, pivot in middle -->
+  <xacro:property name="bogie_length"     value="0.180" />
   <xacro:property name="bogie_width"      value="0.018" />
   <xacro:property name="bogie_height"     value="0.012" />
   <xacro:property name="bogie_mass"       value="0.02"  />
-  <xacro:property name="bogie_half"       value="0.060" />
+  <xacro:property name="bogie_half"       value="0.090" />
   <!-- Differential bar -->
-  <xacro:property name="diff_bar_length"  value="0.200" />
+  <xacro:property name="diff_bar_length"  value="0.300" />
   <xacro:property name="diff_bar_radius"  value="0.005" />
   <xacro:property name="diff_bar_mass"    value="0.02"  />
